File: kicad/evws1/converter-and-cp2.sch (KiCad schematic (older format))
At the start: 50 parts, among them Q4 AO3400, Q5 AO3401, Q6 AO3401, Q7 AO3400, SW6 SS-12D00G3, SW7 SS-12D00G3, U11 PC817C, U12 LM258

Commit message: ...
Parts:
- removed D9: BAT54S, Project:sot-23_hand-soldering, symbol _project:BAT54S
- removed R59, R60: 22k, Project:r-0805-hand-soldering, symbol Device:R
- added C12: 100n, Project:c-1206-hand-soldering, symbol Device:C_Small
- added C47, C48: 1n, Project:c-1206-hand-soldering, symbol Device:C_Small
- added C49, C50: 1u, Project:c-1206-hand-soldering, symbol Device:C_Small
- added D2: LM285M-2.5, Project:SOIC-8_3.9x4.9mm_Pitch1.27mm_Handsolded, symbol _project:LM285M-2.5
- added R18: 10K, Project:r-0805-hand-soldering, symbol Device:R
- added R91, R92: 22K, Project:r-0805-hand-soldering, symbol Device:R
- added R93: 560R, Project:r-0805-hand-soldering, symbol Device:R
Connections:
- net +12V: now also C27.2, U12.8 (V+), C47.1, C50.2
- net +3V3: no longer C27.2, U12.8 (V+)
- net -12V: now also U12.4 (V-), C48.1, C49.2
- net GND: now also U12.5 (+), C12.1, C49.1, C50.1, D2.4 (A); no longer U12.4 (V-)
- net VCP: now also R93.1; no longer C28.1, D11.1 (K), R61.1, U12.2 (-)
- net at Q7.1 (G), R48.2, R50.1: now also C48.2
- net at Q6.1 (G), R46.2, R49.1: now also C47.2
- net at U12.6 (-): now also R91.1, R92.2
- net VREF-2V5: now reaches U12.7
- net VREF-2V5: now also R92.1
- new net: C28.1, D11.1 (K), R61.1, R93.2, U12.2 (-)
- new net +5V: R18.2
- new net VREF+2V5: C12.2, D2.8 (K), R18.1, R91.2
Other:
- moved on the sheet: C27, C28, D11, R53, R54, R61, U12A, U12B, U12C
