File: kicad/evws1/converter-and-cp2.sch (KiCad schematic (older format))
At the start: 57 parts, among them Q4 AO3400, Q5 AO3401, Q6 AO3401, Q7 AO3400, SW6 SS-12D00G3, SW7 SS-12D00G3, U11 PC817C, U12 LM258

Commit message: ...
Parts:
- C23: footprint Project:capacitor-ceramic-tht-2200pf-1000v -> Project:c-1206-hand-soldering
- R18, R24, R25, R35, R36, R37, R38, R39, R40, R42, R43, R44, R45, R46, R47, R48, R49, R50, R51, R52, R53, R54, R55, R56, R57, R58, R61, R91, R92, R93: footprint Project:r-0805-hand-soldering -> Project:r-1206-hand-soldering
Connections:
- net +3V3: no longer Q5.2 (S), R47.2
- net +5V: now also Q5.2 (S), R47.2
- net IRQ-IN: now also D8.3
- net IRQ-OUT: no longer D8.3
- net MISO-IN: now also D7.3
- net MISO-OUT: no longer D7.3
Other:
- moved on the sheet: D7, D8, R35, R36, R39, R40, R44, R45

Commit message: ...
Parts:
- removed C27: 100n, Project:c-1206-hand-soldering, symbol Device:C_Small
- added C40, C53: 100n, Project:c-1206-hand-soldering, symbol Device:C_Small
- renumbered R93 to R5
Connections:
- net +12V: now also C40.2
- net -12V: now also C53.1
- net GND: now also C40.1, C53.2
- net CP2 renamed CP
- no-connect marks 3 -> 4
Changed lines of the file:
@@
 PWM2-IN
 Text HLabel 10025 2500 2    50   Output ~ 0
-CP2
+CP
 Text Label 7150 2500 0    50   ~ 0
-CP
+C1
 $Comp
 L Device:R R?
@@
 Wire Wire Line
 	13075 3825 13075 3725
-Wire Wire Line
-	5675 5025 5675 4925
-Wire Wire Line
-	5675 5725 5675 5625
-$Comp
-L Device:C_Small C?
-U 1 1 5E29ECC7
-P 5875 4925
-AR Path="/5E0A3961/5F6ED0C4/5E29ECC7" Ref="C?"  Part="1"
-AR Path="/5E0A3961/5E29AFD8/5E29ECC7" Ref="C27"  Part="1"
-F 0 "C27" V 5646 4925 50  0000 C CNN
-F 1 "100n" V 5737 4925 50  0000 C CNN
-F 2 "Project:c-1206-hand-soldering" H 5875 4925 50  0001 C CNN
-F 3 "~" H 5875 4925 50  0001 C CNN
-	1    5875 4925
-	0    1    1    0
-$EndComp
-Wire Wire Line
-	5775 4925 5675 4925
-Connection ~ 5675 4925
-Wire Wire Line
-	5675 4925 5675 4725
-$Comp
-L power:GND #PWR?
-U 1 1 5E29ECD1
-P 6075 5025
-AR Path="/5E0A3961/5F6ED0C4/5E29ECD1" Ref="#PWR?"  Part="1"
-AR Path="/5E0A3961/5E29AFD8/5E29ECD1" Ref="#PWR0187"  Part="1"
-F 0 "#PWR0187" H 6075 4775 50  0001 C CNN
-F 1 "GND" H 6075 4875 50  0000 C CNN
-F 2 "" H 6075 5025 50  0001 C CNN
-F 3 "" H 6075 5025 50  0001 C CNN
-	1    6075 5025
-	1    0    0    -1
-$EndComp
-Wire Wire Line
-	5975 4925 6075 4925
-Wire Wire Line
-	6075 4925 6075 5025
 Text HLabel 10025 2350 2    50   UnSpc ~ 0
 PE
@@
 	6950 2500 7800 2500
 Connection ~ 8025 2500
-$Comp
-L _project:LM258 U12
-U 1 1 5E2AA288
-P 8400 3700
-F 0 "U12" H 8450 4000 50  0000 C CNN
-F 1 "LM258" H 8475 3900 50  0000 C CNN
-F 2 "Project:soic-8_hand-soldering" H 9850 3800 50  0001 C CNN
-F 3 "" H 9950 3900 50  0001 C CNN
-	1    8400 3700
-	1    0    0    -1
-$EndComp
-$Comp
-L _project:LM258 U12
-U 2 1 5E2AA425
-P 8750 5500
-F 0 "U12" H 8850 5250 50  0000 C CNN
-F 1 "LM258" H 8875 5350 50  0000 C CNN
-F 2 "Project:soic-8_hand-soldering" H 10200 5600 50  0001 C CNN
-F 3 "" H 10300 5700 50  0001 C CNN
-	2    8750 5500
-	1    0    0    1
-$EndComp
-$Comp
-L _project:LM258 U12
-U 3 1 5E2AA88A
-P 5675 5325
-F 0 "U12" H 5733 5371 50  0000 L CNN
-F 1 "LM258" H 5733 5280 50  0000 L CNN
-F 2 "Project:soic-8_hand-soldering" H 7125 5425 50  0001 C CNN
-F 3 "" H 7225 5525 50  0001 C CNN
-	3    5675 5325
-	1    0    0    -1
-$EndComp
 NoConn ~ 10575 5250
 $Comp
@@
 Text Label 9325 5050 0    50   ~ 0
 VREF-2.5V
-$Comp
-L power:-12V #PWR?
-U 1 1 5E451438
-P 5675 5725
-AR Path="/5E451438" Ref="#PWR?"  Part="1"
-AR Path="/5E13857A/5E451438" Ref="#PWR?"  Part="1"
-AR Path="/5E0A3961/5F6ED0C4/5E451438" Ref="#PWR?"  Part="1"
-AR Path="/5E0A3961/5E29AFD8/5E451438" Ref="#PWR0245"  Part="1"
-F 0 "#PWR0245" H 5675 5825 50  0001 C CNN
-F 1 "-12V" H 5690 5898 50  0000 C CNN
-F 2 "" H 5675 5725 50  0001 C CNN
-F 3 "" H 5675 5725 50  0001 C CNN
-	1    5675 5725
-	-1   0    0    1
-$EndComp
-$Comp
-L power:+12V #PWR?
-U 1 1 5E451556
-P 5675 4725
-AR Path="/5E451556" Ref="#PWR?"  Part="1"
-AR Path="/5E13857A/5E451556" Ref="#PWR?"  Part="1"
-AR Path="/5E0A3961/5F6ED0C4/5E451556" Ref="#PWR?"  Part="1"
-AR Path="/5E0A3961/5E29AFD8/5E451556" Ref="#PWR0246"  Part="1"
-F 0 "#PWR0246" H 5675 4575 50  0001 C CNN
-F 1 "+12V" H 5690 4898 50  0000 C CNN
-F 2 "" H 5675 4725 50  0001 C CNN
-F 3 "" H 5675 4725 50  0001 C CNN
-	1    5675 4725
-	1    0    0    -1
-$EndComp
 Wire Wire Line
 	7800 3600 7800 3800
@@
 P 9925 3700
 AR Path="/5E0A3961/5E47E509" Ref="R?"  Part="1"
-AR Path="/5E0A3961/5E29AFD8/5E47E509" Ref="R93"  Part="1"
-F 0 "R93" V 9825 3625 50  0000 C CNN
+AR Path="/5E0A3961/5E29AFD8/5E47E509" Ref="R5"  Part="1"
+F 0 "R5" V 9825 3625 50  0000 C CNN
 F 1 "560R" V 9825 3825 50  0000 C CNN
 F 2 "Project:r-1206-hand-soldering" V 9855 3700 50  0001 C CNN
@@
 	1    0    0    -1
 $EndComp
+NoConn ~ 4750 850
+$Comp
+L Device:C_Small C?
+U 1 1 5E9A529E
+P 5425 4600
+AR Path="/5E0A3961/5E9A529E" Ref="C?"  Part="1"
+AR Path="/5E377C07/5E9A529E" Ref="C?"  Part="1"
+AR Path="/5E0A3961/5E29AFD8/5E9A529E" Ref="C40"  Part="1"
+F 0 "C40" H 5525 4525 50  0000 C CNN
+F 1 "100n" H 5550 4675 50  0000 C CNN
+F 2 "Project:c-1206-hand-soldering" H 5425 4600 50  0001 C CNN
+F 3 "~" H 5425 4600 50  0001 C CNN
+	1    5425 4600
+	-1   0    0    1
+$EndComp
+$Comp
+L power:+12V #PWR?
+U 1 1 5E9A52A5
+P 5725 4350
+AR Path="/5E9A52A5" Ref="#PWR?"  Part="1"
+AR Path="/5E0A3961/5E9A52A5" Ref="#PWR?"  Part="1"
+AR Path="/5E377C07/5E9A52A5" Ref="#PWR?"  Part="1"
+AR Path="/5E0A3961/5E29AFD8/5E9A52A5" Ref="#PWR0186"  Part="1"
+F 0 "#PWR0186" H 5725 4200 50  0001 C CNN
+F 1 "+12V" H 5740 4523 50  0000 C CNN
+F 2 "" H 5725 4350 50  0001 C CNN
+F 3 "" H 5725 4350 50  0001 C CNN
+	1    5725 4350
+	1    0    0    -1
+$EndComp
+$Comp
+L power:-12V #PWR?
+U 1 1 5E9A52AB
+P 5725 5300
+AR Path="/5E9A52AB" Ref="#PWR?"  Part="1"
+AR Path="/5E0A3961/5E9A52AB" Ref="#PWR?"  Part="1"
+AR Path="/5E377C07/5E9A52AB" Ref="#PWR?"  Part="1"
+AR Path="/5E0A3961/5E29AFD8/5E9A52AB" Ref="#PWR0187"  Part="1"
+F 0 "#PWR0187" H 5725 5400 50  0001 C CNN
+F 1 "-12V" H 5740 5473 50  0000 C CNN
+F 2 "" H 5725 5300 50  0001 C CNN
+F 3 "" H 5725 5300 50  0001 C CNN
+	1    5725 5300
+	-1   0    0    1
+$EndComp
+Wire Wire Line
+	5725 5300 5725 5250
+Wire Wire Line
+	5725 4550 5725 4450
+Wire Wire Line
+	5725 4450 5425 4450
+Connection ~ 5725 4450
+Wire Wire Line
+	5725 4450 5725 4350
+Wire Wire Line
+	5425 4450 5425 4500
+$Comp
+L power:GND #PWR?
+U 1 1 5E9A52B7
+P 5075 4950
+AR Path="/5E9A52B7" Ref="#PWR?"  Part="1"
+AR Path="/5E0A3961/5E9A52B7" Ref="#PWR?"  Part="1"
+AR Path="/5E377C07/5E9A52B7" Ref="#PWR?"  Part="1"
+AR Path="/5E0A3961/5E29AFD8/5E9A52B7" Ref="#PWR0188"  Part="1"
+F 0 "#PWR0188" H 5075 4700 50  0001 C CNN
+F 1 "GND" H 5075 4800 50  0000 C CNN
+F 2 "" H 5075 4950 50  0001 C CNN
+F 3 "" H 5075 4950 50  0001 C CNN
+	1    5075 4950
+	1    0    0    -1
+$EndComp
+Wire Wire Line
+	5425 5000 5425 4850
+$Comp
+L Device:C_Small C?
+U 1 1 5E9A52C5
+P 5425 5100
+AR Path="/5E0A3961/5E9A52C5" Ref="C?"  Part="1"
+AR Path="/5E377C07/5E9A52C5" Ref="C?"  Part="1"
+AR Path="/5E0A3961/5E29AFD8/5E9A52C5" Ref="C53"  Part="1"
+F 0 "C53" H 5525 5025 50  0000 C CNN
+F 1 "100n" H 5550 5175 50  0000 C CNN
+F 2 "Project:c-1206-hand-soldering" H 5425 5100 50  0001 C CNN
+F 3 "~" H 5425 5100 50  0001 C CNN
+	1    5425 5100
+	-1   0    0    1
+$EndComp
+Wire Wire Line
+	5425 5200 5425 5250
+Wire Wire Line
+	5425 5250 5725 5250
+Connection ~ 5725 5250
+Wire Wire Line
+	5725 5250 5725 5150
+Wire Wire Line
+	5425 4850 5075 4850
+Wire Wire Line
+	5075 4850 5075 4950
+Connection ~ 5425 4850
+Wire Wire Line
+	5425 4850 5425 4700
+$Comp
+L _project:LM258 U12
+U 1 1 5EA2E3B0
+P 8400 3700
+F 0 "U12" H 8450 4000 50  0000 C CNN
+F 1 "LM258" H 8475 3900 50  0000 C CNN
+F 2 "Project:soic-8_hand-soldering" H 9850 3800 50  0001 C CNN
+F 3 "" H 9950 3900 50  0001 C CNN
+	1    8400 3700
+	1    0    0    -1
+$EndComp
+$Comp
+L _project:LM258 U12
+U 2 1 5EA2E7D2
+P 8750 5500
+F 0 "U12" H 8825 5275 50  0000 C CNN
+F 1 "LM258" H 8875 5350 50  0000 C CNN
+F 2 "Project:soic-8_hand-soldering" H 10200 5600 50  0001 C CNN
+F 3 "" H 10300 5700 50  0001 C CNN
+	2    8750 5500
+	1    0    0    1
+$EndComp
+$Comp
+L _project:LM258 U12
+U 3 1 5EA39C44
+P 5725 4850
+F 0 "U12" H 5875 4800 50  0000 C CNN
+F 1 "LM258" H 5925 4900 50  0000 C CNN
+F 2 "Project:soic-8_hand-soldering" H 7175 4950 50  0001 C CNN
+F 3 "" H 7275 5050 50  0001 C CNN
+	3    5725 4850
+	1    0    0    -1
+$EndComp

Commit message: schematic finished, placement finished
Changed lines of the file:
@@
 Wire Wire Line
 	9625 1600 9625 1700
-$Comp
-L power:+3V3 #PWR?
-U 1 1 5E29ECA1
-P 13075 3025
-AR Path="/5E29ECA1" Ref="#PWR?"  Part="1"
-AR Path="/5E13857A/5E29ECA1" Ref="#PWR?"  Part="1"
-AR Path="/5E0A3961/5F6ED0C4/5E29ECA1" Ref="#PWR?"  Part="1"
-AR Path="/5E0A3961/5E29AFD8/5E29ECA1" Ref="#PWR0183"  Part="1"
-F 0 "#PWR0183" H 13075 2875 50  0001 C CNN
-F 1 "+3V3" H 13090 3198 50  0000 C CNN
-F 2 "" H 13075 3025 50  0001 C CNN
-F 3 "" H 13075 3025 50  0001 C CNN
-	1    13075 3025
-	1    0    0    -1
-$EndComp
-Wire Wire Line
-	13075 3025 13075 3125
-$Comp
-L power:GND #PWR?
-U 1 1 5E29ECAB
-P 13075 3825
-AR Path="/5E0A3961/5F6ED0C4/5E29ECAB" Ref="#PWR?"  Part="1"
-AR Path="/5E0A3961/5E29AFD8/5E29ECAB" Ref="#PWR0184"  Part="1"
-F 0 "#PWR0184" H 13075 3575 50  0001 C CNN
-F 1 "GND" H 13075 3675 50  0000 C CNN
-F 2 "" H 13075 3825 50  0001 C CNN
-F 3 "" H 13075 3825 50  0001 C CNN
-	1    13075 3825
-	1    0    0    -1
-$EndComp
-Wire Wire Line
-	13075 3825 13075 3725
 Text HLabel 10025 2350 2    50   UnSpc ~ 0
 PE
