File: kicad/evws1/uc.sch (KiCad schematic (older format))
At the start: 76 parts, among them J13 atmega-isp-6, J14 header, J23 header, J24 header, M5 rpi-ev-plc-adapter-v1.0, Q3 AO3400, SW3 SW_Push, SW4 dip-switch-4x2pos-smd-1.27mm, SW5 SS-12D00G3, SW8 dip-switch-4x2pos-smd-1.27mm, U1 atmega324p-20au, U4 PCF8591, U7 DS1307ZN, U8 24LC512, U9 PCF8574, Y1 20MHz, Y4 32768kHz

Commit message: ...
Parts:
- added J26: header, Project:idc-header-1x02-p2.54mm-vertical, symbol Connector_Generic:Conn_01x02
- BT1: footprint Project:knob-battery-holder-horizontal-tht -> Project:knob-battery-holder-vertical-tht
- R100, R101, R102, R103, R104, R105, R19, R20, R21, R22, R23, R26, R27, R28, R29, R30, R31, R32, R33, R34, R64, R65, R66, R67, R68, R69, R70, R71, R98, R99: footprint Project:r-0805-hand-soldering -> Project:r-1206-hand-soldering
- SW3: footprint Buttons_Switches_SMD:SW_SPST_FSMSM -> Project:push-button-smd-4.5x4.5mm-black
- gave numbers to parts that had none: 1
Connections:
- wire segments 425 -> 428

Commit message: ...
Parts:
- removed TP2: TestPoint, Wire_Pads:SolderWirePad_single_0-8mmDrill, symbol Connector:TestPoint
- added R106: 0R, Project:r-1206-hand-soldering, symbol Device:R
- TP3: footprint Wire_Pads:SolderWirePad_single_0-8mmDrill -> Measurement_Points:Measurement_Point_Round-TH_Small
Connections:
- wire segments 428 -> 432
- no-connect marks 22 -> 24
Other:
- moved on the sheet: J13, J25, R33, R34, SW4A, SW4B, SW4C, SW4D, SW8A, SW8B, SW8C, SW8D

Commit message: schematic finished, placement finished
Parts:
- removed TP7: TestPoint, Measurement_Points:Measurement_Point_Round-TH_Small, symbol Connector:TestPoint
- added JP1: Jumper_3_Bridged12, Project:idc-header-1x03-p2.54mm-vertical, symbol Jumper:Jumper_3_Bridged12
Connections:
- net labels added: VE1
- wire segments 432 -> 437
Other:
- moved on the sheet: D20, J23, R103
Changed lines of the file:
@@
 Text Label 6600 5350 0    50   ~ 0
 CONNECTED1
-Text Label 4525 6600 0    50   ~ 0
+Text Label 3600 7400 0    50   ~ 0
 DEBUG
 Wire Wire Line
@@
 	1950 7400 2025 7400
 Wire Wire Line
-	2325 7400 4425 7400
+	2325 7400 3400 7400
 $Comp
 L Device:LED D?
 U 1 1 5F025E0E
-P 5150 6825
+P 4100 7550
 AR Path="/5F025E0E" Ref="D?"  Part="1"
 AR Path="/5E0A3961/5F025E0E" Ref="D20"  Part="1"
-F 0 "D20" H 5150 6725 50  0000 C CNN
-F 1 "LED" H 5142 6661 50  0001 C CNN
-F 2 "LEDs:LED_0805_HandSoldering" H 5150 6825 50  0001 C CNN
-F 3 "~" H 5150 6825 50  0001 C CNN
-F 4 "green" H 5150 6925 50  0000 C CNN "color"
-	1    5150 6825
+F 0 "D20" H 4100 7450 50  0000 C CNN
+F 1 "LED" H 4092 7386 50  0001 C CNN
+F 2 "LEDs:LED_0805_HandSoldering" H 4100 7550 50  0001 C CNN
+F 3 "~" H 4100 7550 50  0001 C CNN
+F 4 "green" H 4100 7650 50  0000 C CNN "color"
+	1    4100 7550
 	-1   0    0    1
 $EndComp
@@
 L power:GND #PWR?
 U 1 1 5F025E15
-P 5400 6975
+P 4350 7600
 AR Path="/5F025E15" Ref="#PWR?"  Part="1"
 AR Path="/5E0A3961/5F025E15" Ref="#PWR0261"  Part="1"
-F 0 "#PWR0261" H 5400 6725 50  0001 C CNN
-F 1 "GND" H 5405 6802 50  0000 C CNN
-F 2 "" H 5400 6975 50  0001 C CNN
-F 3 "" H 5400 6975 50  0001 C CNN
-	1    5400 6975
-	1    0    0    -1
-$EndComp
-Wire Wire Line
-	5300 6825 5400 6825
+F 0 "#PWR0261" H 4350 7350 50  0001 C CNN
+F 1 "GND" H 4350 7450 50  0000 C CNN
+F 2 "" H 4350 7600 50  0001 C CNN
+F 3 "" H 4350 7600 50  0001 C CNN
+	1    4350 7600
+	1    0    0    -1
+$EndComp
+Wire Wire Line
+	4250 7550 4350 7550
 $Comp
 L Device:R R?
 U 1 1 5F025E1C
-P 4750 6825
+P 3700 7550
 AR Path="/5F025E1C" Ref="R?"  Part="1"
 AR Path="/5E0A3961/5F025E1C" Ref="R103"  Part="1"
-F 0 "R103" V 4850 6725 50  0000 C CNN
-F 1 "1K" V 4850 6975 50  0000 C CNN
-F 2 "Project:r-1206-hand-soldering" V 4680 6825 50  0001 C CNN
-F 3 "~" H 4750 6825 50  0001 C CNN
-	1    4750 6825
+F 0 "R103" V 3800 7450 50  0000 C CNN
+F 1 "1K" V 3800 7700 50  0000 C CNN
+F 2 "Project:r-1206-hand-soldering" V 3630 7550 50  0001 C CNN
+F 3 "~" H 3700 7550 50  0001 C CNN
+	1    3700 7550
 	0    1    1    0
 $EndComp
 Wire Wire Line
-	4900 6825 5000 6825
-Wire Wire Line
-	5400 6825 5400 6975
+	3850 7550 3950 7550
+Wire Wire Line
+	4350 7550 4350 7600
 $Comp
 L Connector_Generic:Conn_01x02 J23
 U 1 1 5F15C743
-P 4825 7250
-F 0 "J23" H 4850 7050 50  0000 C CNN
-F 1 "header" H 4850 7350 50  0000 C CNN
-F 2 "Project:idc-header-1x02-p2.54mm-vertical" H 4825 7250 50  0001 C CNN
-F 3 "~" H 4825 7250 50  0001 C CNN
-	1    4825 7250
+P 4900 7350
+F 0 "J23" H 4925 7150 50  0000 C CNN
+F 1 "header" H 4925 7450 50  0000 C CNN
+F 2 "Project:idc-header-1x02-p2.54mm-vertical" H 4900 7350 50  0001 C CNN
+F 3 "~" H 4900 7350 50  0001 C CNN
+	1    4900 7350
 	1    0    0    1
 $EndComp
 Wire Wire Line
-	4625 7150 4425 7150
+	4700 7250 4500 7250
 $Comp
 L power:GND #PWR?
 U 1 1 5F1AB5D4
-P 4575 7300
+P 4650 7400
 AR Path="/5F1AB5D4" Ref="#PWR?"  Part="1"
 AR Path="/5E0A3961/5F1AB5D4" Ref="#PWR0262"  Part="1"
-F 0 "#PWR0262" H 4575 7050 50  0001 C CNN
-F 1 "GND" H 4580 7127 50  0000 C CNN
-F 2 "" H 4575 7300 50  0001 C CNN
-F 3 "" H 4575 7300 50  0001 C CNN
-	1    4575 7300
-	1    0    0    -1
-$EndComp
-Wire Wire Line
-	4625 7250 4575 7250
-Wire Wire Line
-	4575 7250 4575 7300
-Wire Wire Line
-	4300 6600 4425 6600
-Wire Wire Line
-	4425 6600 4425 6825
-Wire Wire Line
-	4425 6825 4600 6825
-Connection ~ 4425 6825
-Connection ~ 4425 7150
-Wire Wire Line
-	4425 7150 4425 7400
-Wire Wire Line
-	4425 6825 4425 7150
+F 0 "#PWR0262" H 4650 7150 50  0001 C CNN
+F 1 "GND" H 4655 7227 50  0000 C CNN
+F 2 "" H 4650 7400 50  0001 C CNN
+F 3 "" H 4650 7400 50  0001 C CNN
+	1    4650 7400
+	1    0    0    -1
+$EndComp
+Wire Wire Line
+	4700 7350 4650 7350
+Wire Wire Line
+	4650 7350 4650 7400
 $Comp
 L Device:R R?
@@
 $EndComp
 Wire Wire Line
-	4425 6600 5700 6600
-Connection ~ 4425 6600
-Wire Wire Line
 	6000 6600 6100 6600
 $Comp
@@
 Wire Wire Line
 	5400 1225 5400 1200
-$Comp
-L Connector:TestPoint TP?
-U 1 1 5E47C985
-P 8900 1100
-AR Path="/5E47C985" Ref="TP?"  Part="1"
-AR Path="/5E0A3961/5E47C985" Ref="TP7"  Part="1"
-F 0 "TP7" H 8850 1300 50  0000 L CNN
-F 1 "TestPoint" H 8958 1129 50  0001 L CNN
-F 2 "Measurement_Points:Measurement_Point_Round-TH_Small" H 9100 1100 50  0001 C CNN
-F 3 "~" H 9100 1100 50  0001 C CNN
-	1    8900 1100
-	1    0    0    -1
-$EndComp
-Wire Wire Line
-	8900 1200 8900 1100
-Wire Wire Line
-	8450 1200 8900 1200
+Wire Wire Line
+	8450 1200 8725 1200
 Connection ~ 10775 4650
 Connection ~ 10775 4750
@@
 Wire Wire Line
 	10500 2050 10500 2450
+Text HLabel 8725 1200 2    50   Output ~ 0
+AOUT
+Text HLabel 4650 6300 2    50   Input ~ 0
+VE1
+$Comp
+L Jumper:Jumper_3_Bridged12 JP1
+U 1 1 5F30065F
+P 4500 6600
+F 0 "JP1" V 4546 6667 50  0000 L CNN
+F 1 "Jumper_3_Bridged12" V 4455 6667 50  0000 L CNN
+F 2 "Project:idc-header-1x03-p2.54mm-vertical" H 4500 6600 50  0001 C CNN
+F 3 "~" H 4500 6600 50  0001 C CNN
+	1    4500 6600
+	0    1    -1   0
+$EndComp
+Connection ~ 4500 7250
+Wire Wire Line
+	4500 7250 4500 7400
+Wire Wire Line
+	4500 6850 4500 7000
+Wire Wire Line
+	4350 6600 4300 6600
+Wire Wire Line
+	3550 7550 3400 7550
+Wire Wire Line
+	3400 7550 3400 7400
+Connection ~ 3400 7400
+Wire Wire Line
+	3400 7400 4500 7400
+Wire Wire Line
+	5700 6600 5550 6600
+Wire Wire Line
+	5550 6600 5550 7000
+Wire Wire Line
+	5550 7000 4500 7000
+Connection ~ 4500 7000
+Wire Wire Line
+	4500 7000 4500 7250
+Wire Wire Line
+	4650 6300 4500 6300
+Wire Wire Line
+	4500 6300 4500 6350
 $EndSCHEMATC

Commit message: ...
Connections:
- net labels removed: GNDA
Other:
- moved on the sheet: R65
Changed lines of the file:
@@
 Wire Wire Line
 	1350 2100 975  2100
-Text Label 1000 1750 0    50   ~ 0
+Text Label 1025 2100 0    50   ~ 0
 ~RESET1
-Text Label 1000 2100 0    50   ~ 0
+Text Label 1025 1750 0    50   ~ 0
 ~RESET2
 Wire Wire Line
@@
 Text Label 8475 1400 0    50   ~ 0
 VREF
-$Comp
-L power:GNDA #PWR0160
-U 1 1 5E758D7C
-P 8675 1875
-F 0 "#PWR0160" H 8675 1625 50  0001 C CNN
-F 1 "GNDA" H 8680 1702 50  0000 C CNN
-F 2 "" H 8675 1875 50  0001 C CNN
-F 3 "" H 8675 1875 50  0001 C CNN
-	1    8675 1875
-	1    0    0    -1
-$EndComp
 Wire Wire Line
 	8450 1800 8675 1800
@@
 	10250 3450 10850 3450
 Wire Wire Line
-	10500 3550 10850 3550
-Wire Wire Line
 	10000 3350 10000 3250
 Wire Wire Line
@@
 Wire Wire Line
 	10250 3450 10250 3250
-Wire Wire Line
-	10500 3775 10500 3550
-Wire Wire Line
-	10500 3550 10500 3250
 Wire Wire Line
 	10000 4075 10000 4125
@@
 L Device:R R65
 U 1 1 5EBEEA13
-P 9750 3400
-F 0 "R65" H 9875 3450 50  0000 C CNN
-F 1 "6K8" H 9875 3350 50  0000 C CNN
-F 2 "Project:r-1206-hand-soldering" V 9680 3400 50  0001 C CNN
-F 3 "~" H 9750 3400 50  0001 C CNN
-	1    9750 3400
+P 9750 3350
+F 0 "R65" H 9875 3400 50  0000 C CNN
+F 1 "6K8" H 9875 3300 50  0000 C CNN
+F 2 "Project:r-1206-hand-soldering" V 9680 3350 50  0001 C CNN
+F 3 "~" H 9750 3350 50  0001 C CNN
+	1    9750 3350
 	1    0    0    -1
 $EndComp
@@
 Connection ~ 10000 3350
 Connection ~ 10250 3450
-Connection ~ 10500 3550
 Text Label 10650 3650 0    50   ~ 0
 AIN3
 Wire Wire Line
-	9750 3650 9750 3550
-Wire Wire Line
-	9750 3650 10850 3650
-Wire Wire Line
-	9750 3250 9750 3150
+	9750 3200 9750 3150
 $Comp
 L power:+5V #PWR?
@@
 	5350 4450 5275 4450
 Wire Wire Line
-	9750 3800 9750 3650
-Connection ~ 9750 3650
-Wire Wire Line
 	9100 2850 9150 2850
 Wire Wire Line
@@
 Wire Wire Line
 	4500 6300 4500 6350
+$Comp
+L power:GND #PWR?
+U 1 1 5F85ACEA
+P 8675 1875
+AR Path="/5F85ACEA" Ref="#PWR?"  Part="1"
+AR Path="/5E0A3961/5F85ACEA" Ref="#PWR0160"  Part="1"
+F 0 "#PWR0160" H 8675 1625 50  0001 C CNN
+F 1 "GND" H 8680 1702 50  0000 C CNN
+F 2 "" H 8675 1875 50  0001 C CNN
+F 3 "" H 8675 1875 50  0001 C CNN
+	1    8675 1875
+	1    0    0    -1
+$EndComp
+Wire Wire Line
+	9750 3500 9750 3550
+Wire Wire Line
+	10500 3250 10500 3650
+Wire Wire Line
+	10850 3550 9750 3550
+Connection ~ 9750 3550
+Wire Wire Line
+	9750 3550 9750 3800
+Wire Wire Line
+	10850 3650 10500 3650
+Connection ~ 10500 3650
+Wire Wire Line
+	10500 3650 10500 3775
 $EndSCHEMATC

Commit message: ...
Parts:
- renumbered J25 to J15, J23 to T5
Changed lines of the file:
@@
 	4350 7550 4350 7600
 $Comp
-L Connector_Generic:Conn_01x02 J23
+L Connector_Generic:Conn_01x02 T5
 U 1 1 5F15C743
 P 4900 7350
-F 0 "J23" H 4925 7150 50  0000 C CNN
+F 0 "T5" H 4925 7150 50  0000 C CNN
 F 1 "header" H 4925 7450 50  0000 C CNN
 F 2 "Project:idc-header-1x02-p2.54mm-vertical" H 4900 7350 50  0001 C CNN
@@
 NoConn ~ 9100 4450
 $Comp
-L Connector_Generic:Conn_01x04 J25
+L Connector_Generic:Conn_01x04 J15
 U 1 1 5FF59D61
 P 10850 2450
-F 0 "J25" H 10875 2150 50  0000 C CNN
+F 0 "J15" H 10875 2150 50  0000 C CNN
 F 1 "header" H 10875 2650 50  0000 C CNN
 F 2 "Project:idc-header-1x04-p2.54mm-vertical" H 10850 2450 50  0001 C CNN

Commit message: V1.0 Design finished
Parts:
- removed J24: header, Project:idc-header-1x03-p2.54mm-vertical, symbol Connector_Generic:Conn_01x03
- added JP9: header, Project:idc-header-1x03-p2.54mm-vertical, symbol Connector_Generic:Conn_01x03
- added T6: header, Project:idc-header-1x04-p2.54mm-vertical, symbol Connector_Generic:Conn_01x04
- renumbered J26 to J15, J15 to LCD2, D20 to LED1, M5 to M4, TP3 to T7
Connections:
- net labels added: LCD1-BL, PB0, PB1
- wire segments 437 -> 441
Other:
- moved on the sheet: LED1, R103
Changed lines of the file:
@@
 encoding utf-8
 Sheet 3 5
-Title ""
-Date ""
-Rev ""
-Comp ""
-Comment1 ""
+Title "Electro Vehicle Wallbox Station"
+Date "2020-02-23"
+Rev "V1.0"
+Comp "(C) Manfred Steiner"
+Comment1 "https://github.com/greenenergyprojects/electro-vehicle-wallbox-station/evws1"
 Comment2 ""
 Comment3 ""
@@
 $EndComp
 $Comp
-L _project:rpi-ev-plc-adapter-v1.0 M5
+L _project:rpi-ev-plc-adapter-v1.0 M4
 U 1 1 5E152A84
 P 8100 4600
-F 0 "M5" H 7325 6500 50  0000 C CNN
+F 0 "M4" H 7325 6500 50  0000 C CNN
 F 1 "rpi-ev-plc-adapter-v1.0" H 8450 6525 50  0000 C CNN
 F 2 "Project:rpi-ev-plc-adapter-v1.0" H 8100 4650 50  0001 C CIN
@@
 Wire Wire Line
 	4350 1450 4300 1450
-Wire Wire Line
-	4300 2250 4750 2250
 Text Notes 4900 2075 0    50   ~ 0
 Slave Address\n1101000
@@
 Wire Wire Line
 	6450 2250 6450 2050
-Connection ~ 4750 2250
 Text Notes 8000 2150 0    50   ~ 0
 Slave Address\n(1001XXX)\n1001001
@@
 Text Label 6600 5350 0    50   ~ 0
 CONNECTED1
-Text Label 3600 7400 0    50   ~ 0
+Text Label 5150 7000 0    50   ~ 0
 DEBUG
 Wire Wire Line
@@
 Wire Wire Line
 	1950 7400 2025 7400
-Wire Wire Line
-	2325 7400 3400 7400
 $Comp
 L Device:LED D?
 U 1 1 5F025E0E
-P 4100 7550
+P 3375 7450
 AR Path="/5F025E0E" Ref="D?"  Part="1"
-AR Path="/5E0A3961/5F025E0E" Ref="D20"  Part="1"
-F 0 "D20" H 4100 7450 50  0000 C CNN
-F 1 "LED" H 4092 7386 50  0001 C CNN
-F 2 "LEDs:LED_0805_HandSoldering" H 4100 7550 50  0001 C CNN
-F 3 "~" H 4100 7550 50  0001 C CNN
-F 4 "green" H 4100 7650 50  0000 C CNN "color"
-	1    4100 7550
-	-1   0    0    1
+AR Path="/5E0A3961/5F025E0E" Ref="LED1"  Part="1"
+F 0 "LED1" H 3375 7350 50  0000 C CNN
+F 1 "LED" H 3367 7286 50  0001 C CNN
+F 2 "LEDs:LED_0805_HandSoldering" H 3375 7450 50  0001 C CNN
+F 3 "~" H 3375 7450 50  0001 C CNN
+F 4 "green" H 3375 7550 50  0000 C CNN "color"
+	1    3375 7450
+	1    0    0    1
 $EndComp
 $Comp
 L power:GND #PWR?
 U 1 1 5F025E15
-P 4350 7600
+P 3125 7450
 AR Path="/5F025E15" Ref="#PWR?"  Part="1"
 AR Path="/5E0A3961/5F025E15" Ref="#PWR0261"  Part="1"
-F 0 "#PWR0261" H 4350 7350 50  0001 C CNN
-F 1 "GND" H 4350 7450 50  0000 C CNN
-F 2 "" H 4350 7600 50  0001 C CNN
-F 3 "" H 4350 7600 50  0001 C CNN
-	1    4350 7600
-	1    0    0    -1
-$EndComp
-Wire Wire Line
-	4250 7550 4350 7550
+F 0 "#PWR0261" H 3125 7200 50  0001 C CNN
+F 1 "GND" H 3125 7300 50  0000 C CNN
+F 2 "" H 3125 7450 50  0001 C CNN
+F 3 "" H 3125 7450 50  0001 C CNN
+	1    3125 7450
+	1    0    0    -1
+$EndComp
 $Comp
 L Device:R R?
 U 1 1 5F025E1C
-P 3700 7550
+P 3750 7450
 AR Path="/5F025E1C" Ref="R?"  Part="1"
 AR Path="/5E0A3961/5F025E1C" Ref="R103"  Part="1"
-F 0 "R103" V 3800 7450 50  0000 C CNN
-F 1 "1K" V 3800 7700 50  0000 C CNN
-F 2 "Project:r-1206-hand-soldering" V 3630 7550 50  0001 C CNN
-F 3 "~" H 3700 7550 50  0001 C CNN
-	1    3700 7550
-	0    1    1    0
-$EndComp
-Wire Wire Line
-	3850 7550 3950 7550
-Wire Wire Line
-	4350 7550 4350 7600
-$Comp
-L Connector_Generic:Conn_01x02 T5
-U 1 1 5F15C743
-P 4900 7350
-F 0 "T5" H 4925 7150 50  0000 C CNN
-F 1 "header" H 4925 7450 50  0000 C CNN
-F 2 "Project:idc-header-1x02-p2.54mm-vertical" H 4900 7350 50  0001 C CNN
-F 3 "~" H 4900 7350 50  0001 C CNN
-	1    4900 7350
-	1    0    0    1
-$EndComp
-Wire Wire Line
-	4700 7250 4500 7250
+F 0 "R103" V 3850 7550 50  0000 C CNN
+F 1 "1K" V 3850 7350 50  0000 C CNN
+F 2 "Project:r-1206-hand-soldering" V 3680 7450 50  0001 C CNN
+F 3 "~" H 3750 7450 50  0001 C CNN
+	1    3750 7450
+	0    -1   -1   0
+$EndComp
 $Comp
 L power:GND #PWR?
 U 1 1 5F1AB5D4
-P 4650 7400
+P 4650 7350
 AR Path="/5F1AB5D4" Ref="#PWR?"  Part="1"
 AR Path="/5E0A3961/5F1AB5D4" Ref="#PWR0262"  Part="1"
-F 0 "#PWR0262" H 4650 7150 50  0001 C CNN
-F 1 "GND" H 4655 7227 50  0000 C CNN
-F 2 "" H 4650 7400 50  0001 C CNN
-F 3 "" H 4650 7400 50  0001 C CNN
-	1    4650 7400
-	1    0    0    -1
-$EndComp
-Wire Wire Line
-	4700 7350 4650 7350
-Wire Wire Line
-	4650 7350 4650 7400
+F 0 "#PWR0262" H 4650 7100 50  0001 C CNN
+F 1 "GND" H 4655 7177 50  0000 C CNN
+F 2 "" H 4650 7350 50  0001 C CNN
+F 3 "" H 4650 7350 50  0001 C CNN
+	1    4650 7350
+	1    0    0    -1
+$EndComp
+Wire Wire Line
+	4700 7250 4650 7250
+Wire Wire Line
+	4650 7250 4650 7350
 $Comp
 L Device:R R?
@@
 Connection ~ 5500 3250
 $Comp
-L Connector_Generic:Conn_01x03 J24
-U 1 1 5FB2E3D2
-P 4550 2650
-F 0 "J24" V 4550 2950 50  0000 R CNN
-F 1 "header" V 4650 2775 50  0000 R CNN
-F 2 "Project:idc-header-1x03-p2.54mm-vertical" H 4550 2650 50  0001 C CNN
-F 3 "~" H 4550 2650 50  0001 C CNN
-	1    4550 2650
-	0    -1   -1   0
-$EndComp
-$Comp
 L power:GND #PWR?
 U 1 1 5FB880F9
-P 4450 2900
+P 4350 2900
 AR Path="/5FB880F9" Ref="#PWR?"  Part="1"
 AR Path="/5E0A3961/5FB880F9" Ref="#PWR0264"  Part="1"
-F 0 "#PWR0264" H 4450 2650 50  0001 C CNN
-F 1 "GND" H 4450 2750 50  0000 C CNN
-F 2 "" H 4450 2900 50  0001 C CNN
-F 3 "" H 4450 2900 50  0001 C CNN
-	1    4450 2900
-	1    0    0    -1
-$EndComp
-Wire Wire Line
-	4450 2850 4450 2900
-Wire Wire Line
-	4300 3150 4550 3150
+F 0 "#PWR0264" H 4350 2650 50  0001 C CNN
+F 1 "GND" H 4350 2750 50  0000 C CNN
+F 2 "" H 4350 2900 50  0001 C CNN
+F 3 "" H 4350 2900 50  0001 C CNN
+	1    4350 2900
+	1    0    0    -1
+$EndComp
 Wire Wire Line
 	4850 3150 4850 2850
 Wire Wire Line
 	4850 2850 5250 2850
-Wire Wire Line
-	4550 2850 4550 3150
-Connection ~ 4550 3150
-Wire Wire Line
-	4550 3150 4850 3150
 Wire Wire Line
 	4300 3250 4650 3250
@@
 Connection ~ 10500 1900
 $Comp
-L Connector_Generic:Conn_01x02 J26
+L Connector_Generic:Conn_01x02 J15
 U 1 1 5E452483
 P 5750 950
-F 0 "J26" H 5775 750 50  0000 C CNN
+F 0 "J15" H 5775 750 50  0000 C CNN
 F 1 "header" H 5725 1050 50  0000 C CNN
 F 2 "Project:idc-header-1x02-p2.54mm-vertical" H 5750 950 50  0001 C CNN
@@
 NoConn ~ 9100 4450
 $Comp
-L Connector_Generic:Conn_01x04 J15
+L Connector_Generic:Conn_01x04 LCD2
 U 1 1 5FF59D61
 P 10850 2450
-F 0 "J15" H 10875 2150 50  0000 C CNN
+F 0 "LCD2" H 10875 2150 50  0000 C CNN
 F 1 "header" H 10875 2650 50  0000 C CNN
 F 2 "Project:idc-header-1x04-p2.54mm-vertical" H 10850 2450 50  0001 C CNN
@@
 P 10550 2050
 AR Path="/5E901354" Ref="TP?"  Part="1"
-AR Path="/5E0A3961/5E901354" Ref="TP3"  Part="1"
-F 0 "TP3" V 10550 2225 50  0000 L CNN
+AR Path="/5E0A3961/5E901354" Ref="T7"  Part="1"
+F 0 "T7" V 10550 2225 50  0000 L CNN
 F 1 "TestPoint" H 10608 2079 50  0001 L CNN
 F 2 "Measurement_Points:Measurement_Point_Round-TH_Small" H 10750 2050 50  0001 C CNN
@@
 	0    1    -1   0
 $EndComp
-Connection ~ 4500 7250
-Wire Wire Line
-	4500 7250 4500 7400
 Wire Wire Line
 	4500 6850 4500 7000
@@
 	4350 6600 4300 6600
 Wire Wire Line
-	3550 7550 3400 7550
-Wire Wire Line
-	3400 7550 3400 7400
-Connection ~ 3400 7400
-Wire Wire Line
-	3400 7400 4500 7400
-Wire Wire Line
 	5700 6600 5550 6600
 Wire Wire Line
@@
 Wire Wire Line
 	5550 7000 4500 7000
-Connection ~ 4500 7000
-Wire Wire Line
-	4500 7000 4500 7250
 Wire Wire Line
 	4650 6300 4500 6300
@@
 Wire Wire Line
 	10500 3650 10500 3775
+Wire Wire Line
+	4500 7000 4500 7150
+Wire Wire Line
+	4500 7150 4700 7150
+Connection ~ 4500 7000
+Wire Wire Line
+	4050 7450 3900 7450
+Wire Wire Line
+	3600 7450 3525 7450
+Wire Wire Line
+	3225 7450 3125 7450
+Wire Wire Line
+	2325 7400 2800 7400
+$Comp
+L Connector_Generic:Conn_01x02 T5
+U 1 1 5E63ECCB
+P 4900 7250
+F 0 "T5" H 5050 7200 50  0000 C CNN
+F 1 "header" H 4900 7350 50  0000 C CNN
+F 2 "Project:idc-header-1x02-p2.54mm-vertical" H 4900 7250 50  0001 C CNN
+F 3 "~" H 4900 7250 50  0001 C CNN
+	1    4900 7250
+	1    0    0    1
+$EndComp
+Text Label 4950 2850 0    50   ~ 0
+PB0
+Text Label 4950 3150 0    50   ~ 0
+PB1
+Text Label 2400 7400 0    50   ~ 0
+LCD1-BL
+$Comp
+L Connector_Generic:Conn_01x04 T6
+U 1 1 5E73E3E0
+P 4450 2650
+F 0 "T6" V 4450 2900 50  0000 R CNN
+F 1 "header" V 4550 2750 50  0000 R CNN
+F 2 "Project:idc-header-1x04-p2.54mm-vertical" H 4450 2650 50  0001 C CNN
+F 3 "~" H 4450 2650 50  0001 C CNN
+	1    4450 2650
+	0    -1   -1   0
+$EndComp
+Connection ~ 4750 2250
+Wire Wire Line
+	4300 2250 4750 2250
+Wire Wire Line
+	4350 2900 4350 2850
+Text Label 4600 3500 0    50   ~ 0
+LCD1-BL
+Wire Wire Line
+	4300 3150 4450 3150
+Wire Wire Line
+	4550 2850 4550 3500
+Wire Wire Line
+	4550 3500 5000 3500
+Wire Wire Line
+	4450 2850 4450 3150
+Connection ~ 4450 3150
+Wire Wire Line
+	4450 3150 4850 3150
+$Comp
+L Connector_Generic:Conn_01x03 JP9
+U 1 1 5E8A0008
+P 4250 7450
+F 0 "JP9" H 4200 7650 50  0000 L CNN
+F 1 "header" H 4150 7250 50  0000 L CNN
+F 2 "Project:idc-header-1x03-p2.54mm-vertical" H 4250 7450 50  0001 C CNN
+F 3 "~" H 4250 7450 50  0001 C CNN
+	1    4250 7450
+	1    0    0    -1
+$EndComp
+Wire Wire Line
+	4500 7150 3950 7150
+Wire Wire Line
+	3950 7150 3950 7350
+Wire Wire Line
+	3950 7350 4050 7350
+Connection ~ 4500 7150
+Wire Wire Line
+	4050 7550 3950 7550
+Wire Wire Line
+	3950 7550 3950 7650
+Wire Wire Line
+	3950 7650 3750 7650
+Text Label 3750 7650 0    50   ~ 0
+PB0
 $EndSCHEMATC
