File: kicad/evws1/_saved_converter-and-cp2.sch (KiCad schematic (older format))
At the start: 57 parts, among them Q4 AO3400, Q5 AO3401, Q6 AO3401, Q7 AO3400, SW6 SS-12D00G3, SW7 SS-12D00G3, U11 PC817C, U12 LM258

Commit message: schematic finished
Connections:
- net IRQ-IN: now also D8.3
- net IRQ-OUT: no longer D8.3
- net MISO-IN: now also D7.3
- net MISO-OUT: no longer D7.3
Other:
- moved on the sheet: D7, D8, R35, R36, R39, R40, R44, R45
