File: kicad/evws1/_saved_uc.sch (KiCad schematic (older format))
At the start: 76 parts, among them J13 atmega-isp-6, J14 header, J23 header, J24 header, M5 rpi-ev-plc-adapter-v1.0, Q3 AO3400, SW3 SW_Push, SW4 dip-switch-4x2pos-smd-1.27mm, SW5 SS-12D00G3, SW8 dip-switch-4x2pos-smd-1.27mm, U1 atmega324p-20au, U4 PCF8591, U7 DS1307ZN, U8 24LC512, U9 PCF8574, Y1 20MHz, Y4 32768kHz

Commit message: schematic finished
Parts:
- gave numbers to parts that had none: 1
Changed lines of the file:
@@
 Wire Wire Line
 	10250 4125 10500 4125
-Text Label 10650 3250 0    50   ~ 0
+Text Label 10650 3350 0    50   ~ 0
 AIN0
-Text Label 10650 3350 0    50   ~ 0
+Text Label 10650 3450 0    50   ~ 0
 AIN1
-Text Label 10650 3450 0    50   ~ 0
+Text Label 10650 3550 0    50   ~ 0
 AIN2
 $Comp
@@
 Connection ~ 10250 3450
 Connection ~ 10500 3550
-Text Label 10650 3550 0    50   ~ 0
+Text Label 10650 3650 0    50   ~ 0
 AIN3
 Wire Wire Line
@@
 	10900 1900 10900 1850
 $Comp
-L Connector_Generic:Conn_01x04 J?
+L Connector_Generic:Conn_01x04 J25
 U 1 1 5FF59D61
 P 10850 2350
-F 0 "J?" H 10875 2050 50  0000 C CNN
+F 0 "J25" H 10875 2050 50  0000 C CNN
 F 1 "header" H 10875 2550 50  0000 C CNN
 F 2 "Project:idc-header-1x04-p2.54mm-vertical" H 10850 2350 50  0001 C CNN
@@
 P 10650 2500
 AR Path="/5FF895DD" Ref="#PWR?"  Part="1"
-AR Path="/5E0A3961/5FF895DD" Ref="#PWR?"  Part="1"
-F 0 "#PWR?" H 10650 2250 50  0001 C CNN
+AR Path="/5E0A3961/5FF895DD" Ref="#PWR0265"  Part="1"
+F 0 "#PWR0265" H 10650 2250 50  0001 C CNN
 F 1 "GND" H 10650 2350 50  0000 C CNN
 F 2 "" H 10650 2500 50  0001 C CNN
