File: kicad/evws1/evws1.kicad_pcb (KiCad board)
At the start: 4 copper layers, 112 x 144 mm, 280 parts, among them J1 Screw_Terminal_01x03, J10 Screw_Terminal_01x04, J11 USB 2.0 Mini, J12 USB 2.0 Mini, J13 atmega-isp-6, J14 header, J15 Jumper, J16 header, J17 header, J18 header, J19 header, J2 Screw_Terminal_01x02, J20 header, J21 header, J22 header, J23 header, J24 header, J25 header, J26 header, J3 HB9500-2P, J4 HB9500-3P, J5 Screw_Terminal_01x04, J6 Screw_Terminal_01x03, J7 Screw_Terminal_01x02, J8 HB9500-2P, J9 HB9500-3P, K1 G3MB-202P, K2 G3MB-202P, M1 HLK-PM01, M2 dc-dc-buck-converter-5v-to-3.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, M3 dc-dc-converter-5v-to-p12v-m1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, M5 rpi-ev-plc-adapter-v1.0, Q1 AO3401, Q2 AO3401, Q3 AO3400, Q4 AO3400, Q5 AO3401, Q6 AO3401, Q7 AO3400, SW1 SW_SS13F06-G5, SW2 SW_SS13F06-G5, SW3 SW_Push, SW4 dip-switch-4x2pos-smd-1.27mm, SW5 SS-12D00G3, SW6 SS-12D00G3, SW7 SS-12D00G3, SW8 dip-switch-4x2pos-smd-1.27mm, T1 ZMPT101B, T2 ZMPT101B, U1 atmega324p-20au, U10 max485esa, U11 PC817C, U12 LM258, U13 LM224, U2 ACS712-30, U3 ACS712-30, U4 PCF8591, U5 ch340g, U6 ch340g, U7 DS1307ZN, U8 24LC512, U9 PCF8574, Y1 20MHz, Y2 12MHz, Y3 12MHz, Y4 32768kHz

Commit message: schematic finished, placement finished
Parts:
- removed the H3 at (43.2, 59.6)
- removed TP1, TP2, TP7: TestPoint, Measurement_Points:Measurement_Point_Round-TH_Small
- added C27: 1pF, Project:c-1206-hand-soldering, F.Cu at (94.7, 90.3)
- added C55: 1pF, Project:c-1206-hand-soldering, F.Cu at (105.3, 91.3)
- added C56: 100n, Project:c-1206-hand-soldering, B.Cu at (102.7, 90.2)
- added C57: 100n, Project:c-1206-hand-soldering, B.Cu at (96.8, 90.4)
- added C58: 1u, Project:c-1206-hand-soldering, F.Cu at (100.5, 101.9)
- added C59: 100n, Project:c-1206-hand-soldering, B.Cu at (96.8, 96.9)
- added C60: 100n, Project:c-1206-hand-soldering, B.Cu at (102.7, 96.8)
- added D21: BAT54S, Project:sot-23_hand-soldering, F.Cu at (94.2, 104.0)
- added H8: MountingHole_Pad, Mounting_Holes:MountingHole_2.5mm_Pad_Via, F.Cu at (43.2, 59.6)
- added J27: header, Project:idc-header-1x02-p2.54mm-vertical, F.Cu at (137.5, 80.3)
- added J28: header, Project:idc-header-1x02-p2.54mm-vertical, F.Cu at (47.5, 83.0)
- added JP1: Jumper_3_Bridged12, Project:idc-header-1x03-p2.54mm-vertical, F.Cu at (89.7, 95.1)
- added R107: 1K, Project:r-1206-hand-soldering, F.Cu at (103.2, 107.1)
- added R108: 10K, Project:r-1206-hand-soldering, F.Cu at (92.4, 96.8)
- added R109: 0R, Project:r-1206-hand-soldering, F.Cu at (92.4, 88.9)
- added R110: 0R, Project:r-1206-hand-soldering, F.Cu at (94.7, 96.8)
- added R111: 0R, Project:r-1206-hand-soldering, F.Cu at (106.3, 83.1)
- added R112: 0R, Project:r-1206-hand-soldering, F.Cu at (123.0, 126.4)
- added R113: 10K, Project:r-1206-hand-soldering, F.Cu at (100.6, 86.3)
- added R114: 10K, Project:r-1206-hand-soldering, F.Cu at (90.1, 90.1)
- added R115: 10K, Project:r-1206-hand-soldering, F.Cu at (117.6, 83.1)
- added R116: 470K, Project:r-1206-hand-soldering, F.Cu at (105.3, 100.5)
- added R117: 1K, Project:r-1206-hand-soldering, F.Cu at (100.5, 104.3)
- added U14: LM258, Project:soic-8_hand-soldering, F.Cu at (100.1, 96.8)
- added U15: AD633AR, Project:soic-8_hand-soldering, F.Cu at (100.1, 90.2)
- C13, C18, C38, D11, U7: moved to B.Cu
- C20, D7, D8, R24, R25, R26, R27, R28, R30, R31, R32, R33, R34, R36, R45, R65, R66, R67, R68, R69, R71, U4, U9: moved to F.Cu
- moved R75 129.8 mm to (97.9, 73.7)
- moved R74 129.4 mm to (100.2, 73.7)
- moved R73 129.2 mm to (102.5, 73.7)
- moved R63 129.1 mm to (104.8, 73.7)
- moved Y4 117.7 mm to (109.6, 67.2), turned to 90 degrees
- moved R44 117.4 mm to (94.0, 140.1), turned to 270 degrees
- moved D7 115.4 mm to (93.9, 129.6), turned to 180 degrees
- moved R45 114.5 mm to (87.6, 124.7)
- moved D8 113.7 mm to (87.3, 129.6), turned to 0 degrees
- moved U7 112.6 mm to (110.9, 72.7), turned to 270 degrees
- moved C18 107.9 mm to (107.1, 73.1), turned to 270 degrees
- moved R27 96.7 mm to (127.3, 83.3), turned to 270 degrees
- moved R28 93.1 mm to (132.8, 86.0), turned to 270 degrees
- moved TP3 92.4 mm to (72.9, 116.0)
- moved R29 90.9 mm to (85.2, 91.5)
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- renumbered H8 to H3
Connections:
- H3 pad 1: Net-(H8-Pad1) -> PE
- J2 pad 1: /K1-A1 -> /K1-A2
- J2 pad 2: /K1-A2 -> /K1-A1
- J7 pad 1: /K2-A2 -> /K2-A1
- J7 pad 2: /K2-A1 -> /K2-A2
- U1 pad 30: /Microcontroller/DEBUG -> Net-(JP1-Pad2)
- U4 pad 15: /Microcontroller/AOUT -> /Measurement/AOUT
Routing:
- net /K2-A2: track 15.5 -> 31.9 mm
- net /L-EV2: track 1.74 -> 11.2 mm
- net /L-EV1: track 0.00 -> 9.50 mm
- net /K2-A1: track 17.3 -> 21.7 mm
- net /K1-A1: track 22.6 -> 20.8 mm
Other:
- board text added: "CP1"
- board text added: "CP2 PLC"
- board text added: "GND"
- board text added: "K1-A1"
- board text added: "K1-A2"
- board text added: "K2-A1"
- board text added: "K2-A2"
- board text added: "L EV1"
- board text added: "L EV2"
- board text added: "L K1"
- board text added: "L K2"
- board text added: "N EV1"
- board text added: "N EV2"
- board text added: "N K1"
- board text added: "N K2"
- board text added: "PE EV1"
- board text added: "PE EV2"
- board text added: "T1"
- board text added: "T2"
- board text added: "~ON1"
- board text added: "~ON2"
- board text removed: "1L"
- board text removed: "2L"
- board text removed: "N-EV1"
- board text removed: "N-EV2"
- board text removed: "N-K1"
- board text removed: "N-K2"

Commit message: ...
Parts:
- C37, C38, D14, D15: moved to F.Cu
- D19: moved to B.Cu
- moved C37 32.0 mm to (100.5, 35.2)
- moved R66 27.6 mm to (122.9, 127.1)
- moved R105 24.3 mm to (100.1, 66.6), turned to 180 degrees
- moved R82 24.0 mm to (98.2, 119.1), turned to 90 degrees
- moved R70 18.2 mm to (117.8, 117.2)
- moved R104 14.4 mm to (90.2, 68.8), turned to 270 degrees
- moved TP3 14.0 mm to (59.5, 112.1)
- moved R5 12.9 mm to (105.5, 110.3)
- moved R64 11.0 mm to (125.0, 109.8)
- moved R106 9.58 mm to (133.5, 85.8), turned to 270 degrees
- moved C35 9.00 mm to (63.9, 53.4), turned to 0 degrees
- moved R63 6.80 mm to (98.0, 73.7)
- moved R16 5.52 mm to (102.0, 163.0)
- moved Y3 4.60 mm to (123.0, 51.3)
- moved C30 4.58 mm to (119.5, 46.6), turned to 90 degrees
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Connections:
- C21 pad 1: GNDA -> GND
- H8 pad 1: Net-(H8-Pad1) -> PE
- J1 pad 1: PE -> 230V-N
- J1 pad 2: 230V-N -> 230V-L
- J1 pad 3: 230V-L -> PE
- J16 pad 2: /Microcontroller/DE1 -> /Microcontroller/UC-TXD0
- J16 pad 3: /Microcontroller/~RE1 -> /Microcontroller/UC-RXD0
- J16 pad 6: /Microcontroller/UC-TXD0 -> /Microcontroller/DE1
- J16 pad 7: /Microcontroller/UC-RXD0 -> /Microcontroller/~RE1
- R64 pad 2: /Microcontroller/AIN3 -> /Microcontroller/AIN2
- R65 pad 2: /Microcontroller/AIN3 -> /Microcontroller/AIN2
- R70 pad 2: /Microcontroller/AIN2 -> /Microcontroller/AIN3
- R71 pad 1: /Microcontroller/AIN2 -> /Microcontroller/AIN3
- RV6 pad 1: /Measurement/I1 -> GND
- RV6 pad 3: GND -> /Measurement/I1
- SW4 pad 6: /Microcontroller/~RESET1 -> /Microcontroller/~RESET2
- SW4 pad 8: /Microcontroller/~RESET2 -> /Microcontroller/~RESET1
- T1 pad 2: /N-EV1 -> /N-K1
- U4 pad 13: GNDA -> GND
Routing:
- net PE: track 0.00 -> 403.9 mm
- net GND: track 0.00 -> 254.3 mm, vias 0 -> 54
- net /EV1X: track 0.00 -> 183.1 mm, vias 0 -> 3
- net /Microcontroller/SCL: track 0.00 -> 168.3 mm, vias 0 -> 3
- net /Microcontroller/SDA: track 0.00 -> 166.1 mm, vias 0 -> 4
- net Net-(J24-Pad3): track 0.00 -> 159.7 mm, vias 0 -> 3
- net Net-(J24-Pad2): track 0.00 -> 156.5 mm, vias 0 -> 3
- net +5V: track 0.00 -> 129.2 mm, vias 0 -> 34
- net +3V3: track 0.00 -> 123.0 mm, vias 0 -> 3
- net /Microcontroller/~RESET2: track 0.00 -> 121.7 mm, vias 0 -> 1
- net /Measurement/VREF+2V5: track 0.00 -> 118.9 mm, vias 0 -> 5
- net /~EV1: track 0.00 -> 107.9 mm, vias 0 -> 2
- net /Microcontroller/UC-TXD0: track 0.00 -> 106.5 mm, vias 0 -> 3
- net /Microcontroller/UC-TXD1: track 0.00 -> 106.3 mm, vias 0 -> 4
- net /Microcontroller/UC-RXD0: track 0.00 -> 103.3 mm, vias 0 -> 3
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- added copper zone on In1.Cu, net +12V
- added copper zone on In1.Cu, net +5V
- added copper zone on In1.Cu, net -12V
- added copper zone on B.Cu, net /N-EV1
- added copper zone on B.Cu, net /N-EV2
- added copper zone on B.Cu, net /N-K1
- added copper zone on B.Cu, net /N-K2
- added copper zone on In2.Cu, net GND
Other:
- net class AC230V-0,5mm: clearance 2 -> 1.2
