File: kicad/evws1/evws1.sch (KiCad schematic (older format))
At the start: 72 parts, among them J1 Screw_Terminal_01x03, J10 Screw_Terminal_01x04, J2 Screw_Terminal_01x02, J21 header, J22 header, J27 header, J28 header, J3 HB9500-2P, J4 HB9500-3P, J5 Screw_Terminal_01x04, J6 Screw_Terminal_01x03, J7 Screw_Terminal_01x02, J8 HB9500-2P, J9 HB9500-3P, K1 G3MB-202P, K2 G3MB-202P, M1 HLK-PM01, M2 dc-dc-buck-converter-5v-to-3.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, M3 dc-dc-converter-5v-to-p12v-m1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, Q1 AO3401, Q2 AO3401, SW1 SW_SS13F06-G5, SW2 SW_SS13F06-G5, T1 ZMPT101B, T2 ZMPT101B, U2 ACS712-30, U3 ACS712-30

Commit message: ...
Parts:
- added J29: header, Project:idc-header-1x02-p2.54mm-vertical, symbol Connector_Generic:Conn_01x02
- renumbered C4 to C30, C5 to C35, K1 to SSR1, K2 to SSR2, J21 to T2, J22 to T4, T1 to TR1, T2 to TR2
Connections:
- wire segments 306 -> 310
Changed lines of the file:
@@
 	4100 1050 4150 1050
 $Comp
-L _project:ZMPT101B T2
+L _project:ZMPT101B TR2
 U 1 1 5DF0A9DC
 P 3850 3000
-F 0 "T2" H 3600 3350 50  0000 C CNN
+F 0 "TR2" H 3600 3350 50  0000 C CNN
 F 1 "ZMPT101B" H 4000 3350 50  0000 C CNN
 F 2 "Project:Transformer-zmpt101b_ebay-121438904988" H 3950 3350 50  0001 C CNN
@@
 PE
 $Comp
-L _project:ZMPT101B T1
+L _project:ZMPT101B TR1
 U 1 1 5E1505EE
 P 7450 3000
-F 0 "T1" H 7700 3350 50  0000 C CNN
+F 0 "TR1" H 7700 3350 50  0000 C CNN
 F 1 "ZMPT101B" H 7275 3350 50  0000 C CNN
 F 2 "Project:Transformer-zmpt101b_ebay-121438904988" H 7550 3350 50  0001 C CNN
@@
 MODBUS-A
 $Comp
-L _project:G3MB-202P K1
+L _project:G3MB-202P SSR1
 U 1 1 5E22B2EB
 P 8900 4650
-F 0 "K1" H 8750 4850 50  0000 C CNN
+F 0 "SSR1" H 8750 4850 50  0000 C CNN
 F 1 "G3MB-202P" H 8925 4450 50  0000 C CNN
 F 2 "Project:SSR_Omron_G3MB-202P" H 8700 4450 50  0001 L CIN
@@
 $EndComp
 $Comp
-L _project:G3MB-202P K2
+L _project:G3MB-202P SSR2
 U 1 1 5E22B4C3
 P 2450 4650
-F 0 "K2" H 2600 4850 50  0000 C CNN
+F 0 "SSR2" H 2600 4850 50  0000 C CNN
 F 1 "G3MB-202P" H 2450 4450 50  0000 C CNN
 F 2 "Project:SSR_Omron_G3MB-202P" H 2250 4450 50  0001 L CIN
@@
 	6700 3650 6700 4050
 $Comp
-L Device:C_Small C5
+L Device:C_Small C35
 U 1 1 5E2D8A37
 P 4550 4050
-F 0 "C5" V 4425 4050 50  0000 C CNN
+F 0 "C35" V 4425 4050 50  0000 C CNN
 F 1 "1n" V 4500 4150 50  0000 C CNN
 F 2 "Project:c-1206-hand-soldering" H 4550 4050 50  0001 C CNN
@@
 Connection ~ 4750 4050
 $Comp
-L Device:C_Small C4
+L Device:C_Small C30
 U 1 1 5E356FF9
 P 6900 4050
-F 0 "C4" V 6775 4050 50  0000 C CNN
+F 0 "C30" V 6775 4050 50  0000 C CNN
 F 1 "1n" V 6850 4150 50  0000 C CNN
 F 2 "Project:c-1206-hand-soldering" H 6900 4050 50  0001 C CNN
@@
 	7050 3200 6075 3200
 $Comp
-L Connector_Generic:Conn_01x04 J21
+L Connector_Generic:Conn_01x04 T2
 U 1 1 5E422024
 P 6950 5250
-F 0 "J21" H 6950 4950 50  0000 C CNN
+F 0 "T2" H 6950 4950 50  0000 C CNN
 F 1 "header" H 6925 5450 50  0000 C CNN
 F 2 "Project:idc-header-1x04-p2.54mm-vertical" H 6950 5250 50  0001 C CNN
@@
 Connection ~ 6400 4950
 $Comp
-L Connector_Generic:Conn_01x04 J22
+L Connector_Generic:Conn_01x04 T4
 U 1 1 5E4E08A3
 P 4425 5250
-F 0 "J22" H 4425 4950 50  0000 C CNN
+F 0 "T4" H 4425 4950 50  0000 C CNN
 F 1 "header" H 4400 5450 50  0000 C CNN
 F 2 "Project:idc-header-1x04-p2.54mm-vertical" H 4425 5250 50  0001 C CNN
@@
 Wire Wire Line
 	1900 1250 2400 1250
+$Comp
+L Connector_Generic:Conn_01x02 J?
+U 1 1 5E536ADA
+P 4450 1850
+AR Path="/5E0A3961/5E536ADA" Ref="J?"  Part="1"
+AR Path="/5E536ADA" Ref="J29"  Part="1"
+F 0 "J29" H 4475 1650 50  0000 C CNN
+F 1 "header" H 4425 1950 50  0000 C CNN
+F 2 "Project:idc-header-1x02-p2.54mm-vertical" H 4450 1850 50  0001 C CNN
+F 3 "~" H 4450 1850 50  0001 C CNN
+	1    4450 1850
+	-1   0    0    1
+$EndComp
+Wire Wire Line
+	4750 1750 4650 1750
+Connection ~ 4750 1750
+Wire Wire Line
+	5200 1950 4750 1950
+Wire Wire Line
+	4750 1950 4750 1850
+Wire Wire Line
+	4750 1850 4650 1850
+Connection ~ 5200 1950
 $EndSCHEMATC

Commit message: V1.0 Design finished
Parts:
- removed T2: header, Project:idc-header-1x04-p2.54mm-vertical, symbol Connector_Generic:Conn_01x04
- added T2: header, Project:idc-header-1x06-p2.54mm-vertical, symbol Connector_Generic:Conn_01x06
- renumbered J27 to J16, J28 to J17, J29 to J18, D4 to LED2, D3 to LED3
Connections:
- net labels added: AD-E1, AD-P1
- wire segments 310 -> 318
Changed lines of the file:
@@
 Sheet 1 5
 Title "Electro Vehicle Wallbox Station"
-Date "2019-12-09"
-Rev "0.1"
+Date "2020-02-23"
+Rev "V1.0"
 Comp "(C) Manfred Steiner"
-Comment1 "Branch master"
+Comment1 "https://github.com/greenenergyprojects/electro-vehicle-wallbox-station/evws1"
 Comment2 "kicad/evws1"
 Comment3 "https://github.com/greenenergyprojects/electro-vehicle-wallbox-station"
@@
 F4 "V1P" I R 6075 2800 50
 F5 "V1N" I R 6075 3200 50
-F6 "I1" I R 6075 3850 50
+F6 "I1" I R 6075 3750 50
 F7 "I2" I L 5275 3850 50
 F8 "AD-V1" O R 6075 4000 50
@@
 F14 "AOUT" I R 6075 4300 50
 F15 "E1" O R 6075 4200 50
+F16 "P1" O R 6075 3900 50
 $EndSheet
 Wire Wire Line
-	7150 3850 6075 3850
+	7150 3850 6400 3850
 Wire Wire Line
 	4300 3850 5275 3850
 $Comp
-L Device:LED D3
+L Device:LED LED3
 U 1 1 5E43026F
 P 9025 5150
-F 0 "D3" H 9025 5050 50  0000 C CNN
+F 0 "LED3" H 9025 5050 50  0000 C CNN
 F 1 "LED" H 9017 4986 50  0001 C CNN
 F 2 "LEDs:LED_0805_HandSoldering" H 9025 5150 50  0001 C CNN
@@
 $EndComp
 $Comp
-L Device:LED D4
+L Device:LED LED2
 U 1 1 5E57B472
 P 2325 5200
-F 0 "D4" H 2325 5100 50  0000 C CNN
+F 0 "LED2" H 2325 5100 50  0000 C CNN
 F 1 "LED" H 2317 5036 50  0001 C CNN
 F 2 "LEDs:LED_0805_HandSoldering" H 2325 5200 50  0001 C CNN
@@
 CP1
 Wire Wire Line
-	6150 5250 6750 5250
-Text Label 6750 5250 2    50   ~ 0
+	6150 5250 6800 5250
+Text Label 6800 5250 2    50   ~ 0
 CP1
 $Comp
@@
 $EndComp
 Wire Wire Line
-	6075 4100 6400 4100
-Wire Wire Line
-	6400 4100 6400 4950
-Wire Wire Line
-	6400 4950 6150 4950
-Wire Wire Line
-	6075 4000 6450 4000
-Wire Wire Line
-	6450 4000 6450 5050
-Wire Wire Line
-	6450 5050 6150 5050
+	6325 4950 6150 4950
+Wire Wire Line
+	6375 5050 6150 5050
 Wire Wire Line
 	5275 4100 4950 4100
@@
 F19 "EV1X" I L 5150 6700 50
 F20 "EV2X" I L 5150 6800 50
-F21 "AOUT" O R 6150 4725 50
+F21 "AOUT" O R 6150 4700 50
 F22 "VE1" I R 6150 4800 50
 $EndSheet
@@
 $EndComp
 Wire Wire Line
-	7375 4750 7100 4750
+	7375 4750 7175 4750
 Connection ~ 7375 4750
 Wire Wire Line
 	7375 4750 7375 4900
-Text Label 7150 4750 0    50   ~ 0
+Text Label 7200 4750 0    50   ~ 0
 ~EV1
 $Comp
@@
 	7050 3200 6075 3200
 $Comp
-L Connector_Generic:Conn_01x04 T2
-U 1 1 5E422024
-P 6950 5250
-F 0 "T2" H 6950 4950 50  0000 C CNN
-F 1 "header" H 6925 5450 50  0000 C CNN
-F 2 "Project:idc-header-1x04-p2.54mm-vertical" H 6950 5250 50  0001 C CNN
-F 3 "~" H 6950 5250 50  0001 C CNN
-	1    6950 5250
-	1    0    0    1
-$EndComp
-$Comp
 L power:GND #PWR0258
 U 1 1 5E43948B
@@
 $EndComp
 Wire Wire Line
-	6750 5350 6675 5350
+	6800 5350 6675 5350
 Wire Wire Line
 	6675 5350 6675 5400
-Connection ~ 6400 4950
+Connection ~ 6325 4950
 $Comp
 L Connector_Generic:Conn_01x04 T4
@@
 Connection ~ 4950 4950
 Wire Wire Line
-	6400 5150 6750 5150
-Wire Wire Line
-	6400 4950 6400 5150
-Wire Wire Line
-	6750 5050 6450 5050
-Connection ~ 6450 5050
+	6325 5150 6800 5150
+Wire Wire Line
+	6325 4950 6325 5150
+Wire Wire Line
+	6800 5050 6375 5050
+Connection ~ 6375 5050
 Text Label 4625 5150 0    50   ~ 0
 AD-I2
 Text Label 4625 5050 0    50   ~ 0
 AD-V2
-Text Label 6750 5150 2    50   ~ 0
+Text Label 6800 5150 2    50   ~ 0
 AD-I1
-Text Label 6750 5050 2    50   ~ 0
+Text Label 6800 5050 2    50   ~ 0
 AD-V1
 $Comp
@@
 P 2200 6150
 AR Path="/5E0A3961/5E20BE9A/5ED2AD37" Ref="J?"  Part="1"
-AR Path="/5ED2AD37" Ref="J27"  Part="1"
-F 0 "J27" V 2200 6225 50  0000 L CNN
+AR Path="/5ED2AD37" Ref="J16"  Part="1"
+F 0 "J16" V 2200 6225 50  0000 L CNN
 F 1 "header" V 2300 5975 50  0000 L CNN
 F 2 "Project:idc-header-1x02-p2.54mm-vertical" H 2200 6150 50  0001 C CNN
@@
 P 2600 6150
 AR Path="/5E0A3961/5E20BE9A/5ED434D8" Ref="J?"  Part="1"
-AR Path="/5ED434D8" Ref="J28"  Part="1"
-F 0 "J28" V 2600 5850 50  0000 L CNN
+AR Path="/5ED434D8" Ref="J17"  Part="1"
+F 0 "J17" V 2600 5850 50  0000 L CNN
 F 1 "header" V 2700 5975 50  0000 L CNN
 F 2 "Project:idc-header-1x02-p2.54mm-vertical" H 2600 6150 50  0001 C CNN
@@
 	2300 6700 1825 6700
 Wire Wire Line
-	6150 4725 6225 4725
-Wire Wire Line
-	6225 4725 6225 4300
+	6150 4700 6225 4700
+Wire Wire Line
+	6225 4700 6225 4300
 Wire Wire Line
 	6225 4300 6075 4300
@@
 P 4450 1850
 AR Path="/5E0A3961/5E536ADA" Ref="J?"  Part="1"
-AR Path="/5E536ADA" Ref="J29"  Part="1"
-F 0 "J29" H 4475 1650 50  0000 C CNN
+AR Path="/5E536ADA" Ref="J18"  Part="1"
+F 0 "J18" H 4475 1650 50  0000 C CNN
 F 1 "header" H 4425 1950 50  0000 C CNN
 F 2 "Project:idc-header-1x02-p2.54mm-vertical" H 4450 1850 50  0001 C CNN
@@
 	4750 1850 4650 1850
 Connection ~ 5200 1950
+Wire Wire Line
+	6400 3850 6400 3750
+Wire Wire Line
+	6400 3750 6075 3750
+Wire Wire Line
+	6375 4000 6375 5050
+Wire Wire Line
+	6325 4100 6325 4950
+$Comp
+L Connector_Generic:Conn_01x06 T2
+U 1 1 5E91D597
+P 7000 5150
+F 0 "T2" H 7000 4750 50  0000 C CNN
+F 1 "header" H 7000 5475 50  0000 C CNN
+F 2 "Project:idc-header-1x06-p2.54mm-vertical" H 7000 5150 50  0001 C CNN
+F 3 "~" H 7000 5150 50  0001 C CNN
+	1    7000 5150
+	1    0    0    1
+$EndComp
+Wire Wire Line
+	6275 4800 6425 4800
+Wire Wire Line
+	6425 4800 6425 4950
+Connection ~ 6275 4800
+Text Label 6800 4950 2    50   ~ 0
+AD-E1
+Text Label 6800 4850 2    50   ~ 0
+AD-P1
+Wire Wire Line
+	6425 4950 6800 4950
+Wire Wire Line
+	6325 4100 6075 4100
+Wire Wire Line
+	6375 4000 6075 4000
+Wire Wire Line
+	6075 3900 6475 3900
+Wire Wire Line
+	6475 3900 6475 4850
+Wire Wire Line
+	6475 4850 6800 4850
 $EndSCHEMATC
